File: Hardware/mPCIe.sch (EAGLE design)
At the start: 78 parts, among them CN1 MINI_PCIE_1759547-1SMD, J1 SIM_PRT-00548, Q1 BSS138, U1 EDISON_CONNECTOR_FULLMOUNTING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, U2 USB2512BQFN, U3 BA33DD0WHFPSMD, U4 FT231XS-U, U5 TPS62065, U6 MAX4995AAUT+, U7 BA15BC0FP-E2, Y1 24.000MHZ 50ppm

Commit message: add revision 0.2 of the schematic; added initial board layout; renumbered components; removed solder jumpers; schematic style considerations
Parts:
- removed C30, C31, C34: 47pF, rcl:C-USC0402K
- removed C32, C33: 0.1uF, rcl:C-USC0402K
- removed C35, C36: 22uF, rcl:C-USC0402K
- removed C37: 0.47uF, rcl:C-USC0402K
- removed C38: 22uF TANT, SparkFun-Capacitors:CAP_POL3528
- removed SJ1, SJ2, SJ3: JUMPER-PAD-2-NC_BY_TRACE, SparkFun-Passives:JUMPER-PAD-2-NC_BY_TRACE
- C1, C3: value 0.1uF -> 22uF
- C10: value 0.1uF -> 18pF
- C11, C8: value DNP -> 47pF
- C13, C5, C6: value DNP -> 0.1uF
- C14: value 4.7uF -> 22uF TANT; device rcl:C-USC0603K -> SparkFun-Capacitors:CAP_POL3528
- C15: value 0.1uF -> 0.47uF
- C16, C18: value 1.0uF/DNP -> 0.1uF
- C17: value 0.1uF -> 22uF TANT; device rcl:C-USC0402K -> SparkFun-Capacitors:CAP_POL3528
- C19: value 18pF -> 0.1uF
- C2: value 0.1uF -> 47pF
- C20: value 18pF -> 4.7uF; device rcl:C-USC0402K -> rcl:C-USC0603K
- C22: value 470uF TANT -> 0.1uF; device SparkFun-Capacitors:CAP_POL3528 -> rcl:C-USC0402K
- C23: value 100uF -> 0.1uF; device SparkFun-Capacitors:CAP_POLE -> rcl:C-USC0402K
- C24: value 0.47uF -> 470uF TANT; device rcl:C-USC0402K -> SparkFun-Capacitors:CAP_POL3528
- C25: value 22uF TANT -> 12pF; device SparkFun-Capacitors:CAP_POL3528 -> rcl:C-USC0402K
- C26: value 12pF -> 100uF; device rcl:C-USC0402K -> SparkFun-Capacitors:CAP_POLE
- C7: value DNP -> 0.47uF
- C9: value 1.0uF/DNP -> 18pF; device rcl:C-USC0603K -> rcl:C-USC0402K
- D1: value Yellow -> BLUE; device SparkFun-LED:LED-YELLOW0603 -> SparkFun-LED:LED-BLUE0603
- D2: value RED -> GREEN; device SparkFun-LED:LED-RED0603 -> SparkFun-LED:LED-GREEN0603
- D3: value BLUE -> RED; device SparkFun-LED:LED-BLUE0603 -> SparkFun-LED:LED-RED0603
- D4: value GREEN -> Yellow; device SparkFun-LED:LED-GREEN0603 -> SparkFun-LED:LED-YELLOW0603
- JP2: value USB-MICROB -> (none); device SparkFun-Connectors:USB-MICROB -> SparkFun-Connectors:USB-ABCONN-11794
- R1: value 1Meg -> 1K; device rcl:R-US_R0603 -> rcl:R-US_R0402
- R11: value 27 -> 100
- R13: value 100 -> 1K
- R15: value 1K -> 12.0K 1%
- R16: value 1K -> 100K
- R17: value 680K -> 100K; device rcl:R-US_R0603 -> rcl:R-US_R0402
- R18: value 120K -> 100K; device rcl:R-US_R0603 -> rcl:R-US_R0402
- R19: value 1K -> 58K; device rcl:R-US_R0603 -> rcl:R-US_R0402
- R2: value 12.0K 1% -> 680K; device rcl:R-US_R0603 -> rcl:R-US_R0402
- R3: value 100K -> 120K; device rcl:R-US_R0603 -> rcl:R-US_R0402
- R4, R6: value 100K -> 1K; device rcl:R-US_R0603 -> rcl:R-US_R0402
- R5, R7: device rcl:R-US_R0603 -> rcl:R-US_R0402
- R8: value 1K -> 1Meg; device rcl:R-US_R0603 -> rcl:R-US_R0402
- R9: value 58K -> 27; device rcl:R-US_R0603 -> rcl:R-US_R0402
- Y1: value 24.000MHZ 50ppm -> 24MHz 50ppm; device SparkFun-FreqCtrl:CRYSTALSMD -> SparkFun-FreqCtrl:CRYSTAL5X3
Connections:
- removed net N$16: SJ1.1, U4.CBUS1
- removed net N$21: R15.2, SJ2.2
- removed net N$30: R19.1, SJ3.2
- removed net OSC_N2: U2.!OSC_N2
- removed net P$1: C38.+, CN1.+1.5V@28, CN1.+1.5V@48, CN1.+1.5V@6, U7.OUT
- removed net USB_UP_DM: U2.USBDM_UP
- new net 1.5V: C17.+, CN1.+1.5V@28, CN1.+1.5V@48, CN1.+1.5V@6, U7.OUT
- net 1.8V: now also C4.1; no longer C32.1
- net 3.3V: now also C16.1, C18.1, C19.1, C20.1, C21.1, C22.1, C23.1, R5.2, R6.2, R7.2; no longer C1.1, C10.1, C11.1, C12.1, C13.1, C14.1, C2.1, C3.1, C4.1, C5.1, C6.1, C7.1, C8.1, C9.1, R3.2, R4.2, R8.2
- net 3.3V_2A: now also C14.+, C24.+; no longer C22.+, C25.+
- net 5V: now also C1.1, C6.1, R1.2; no longer C33.1, C36.1, R16.2
- net GND: now also C10.1, C14.-, C17.-, C19.2, C20.2, C22.2, C23.2, C24.-, C25.2, C26.-, C9.1, JP2.SHIELD, R15.1, R16.1, R17.1, R19.2, R3.1, R4.1; no longer C10.2, C14.2, C17.2, C19.1, C2.2, C20.1, C22.-, C23.-, C24.2, C25.-, C26.2, C30.2, C31.2, C32.2, C33.2, C35.2, C36.2, C37.2, C38.-, C9.2, R2.1, R5.1, R6.1, R7.1, R9.2, SJ3.1
- net N$1: now also C13.1; no longer C15.1, C16.1
- net N$10: now also R16.2; no longer R7.2
- net N$11: now also R9.1; no longer R10.1
- net N$12: now also R17.2; no longer R6.2
- net N$13: now also R10.1; no longer R11.1
- net N$14: now also C8.1, R9.2; no longer C30.1, R10.2
- net N$15: now also C11.1, R10.2; no longer C31.1, R11.2
- net N$17: now also R11.2; no longer R12.2
- net N$18: now also R12.2; no longer R13.2
- net N$19: now also R14.2; no longer SJ2.1
- net N$2: now also C9.2, R8.2, Y1.2; no longer C19.2, R1.2, Y1.1
- net N$20: now also R13.2, U4.CBUS1; no longer R14.2, SJ1.2
- net N$22: now also D3.C, R13.1; no longer D2.C, R14.1
- net N$23: now also D4.C, R14.1; no longer D1.C, R15.1
- net N$24: now also R1.1; no longer R16.1
- net N$26: now also C2.2, R2.1, R3.2; no longer C34.2, R17.1, R18.2
- net N$27: now also R19.1; no longer R9.1
- net N$28: now also D2.A, R6.1; no longer D4.A, R8.1
- net N$29: now also D1.C, R4.2; no longer D3.C, R19.2
- net N$3: now also C12.1; no longer C17.1, C18.1
- net N$4: now also C10.2, R8.1, Y1.1; no longer C20.2, R1.1, Y1.2
- net N$5: now also R15.2; no longer R2.2
- net N$6: now also C5.1, R5.1; no longer C21.1, R3.1
- net N$7: now also D2.C, R7.1; no longer D4.C, R4.1
- net N$8: now also R18.2; no longer R5.2
- net N$9: now also C26.+; no longer C23.+
- net OCS_N2: now also U2.!OCS_N2
- net UART_2_RX: now also R11.1; no longer R12.1
- net UART_2_TX: now also R12.1; no longer R13.1
- net UIM_CLK: now also C25.1; no longer C26.1
- net USB_UP_DN: now also U2.USBDM_UP
- net VSYS: now also C15.1, C2.1, C3.1, C7.1, D4.A, R2.2; no longer C24.1, C34.1, C35.1, C37.1, D2.A, R17.2
Other:
- note added: "----------------------- Revision Notes:"
- note added: "0.2"
- note added: "4v to 1.5v/1A LDO"
- note added: "Changed: crystal footprint; DN_USB to AB; Mov. cap bank; rem. SJ"
- note added: "Each 0.1uF filtering cap should be close to pins 23, 15, 5, 10, 29, 36"
- note added: "Filtering cap for pin 15"
- note added: "JP2"
- note removed: "0.1"
- note removed: "4v to 1.5v/1A LDO (optional)"
- moved on the sheet: C1, C10, C11, C12, C13, C15, C16, C18, C19, C2, C20, C21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

Commit message: moved all components onto layout; grouped by major function
Parts:
- L1: value 1.0uH -> (none)
Changed lines of the file:
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@@
 <part name="SUPPLY2" library="SparkFun-Aesthetics" deviceset="5V" device=""/>
 <part name="GND4" library="SparkFun-Aesthetics" deviceset="GND" device=""/>
-<part name="L1" library="SparkFun-Passives" deviceset="INDUCTOR" device="" value="1.0uH"/>
+<part name="L1" library="SparkFun-Passives" deviceset="INDUCTOR" device=""/>
 <part name="R2" library="rcl" deviceset="R-US_" device="R0402" value="680K"/>
 <part name="R3" library="rcl" deviceset="R-US_" device="R0402" value="120K"/>

Commit message: v0.3 of schematic: connected all the 3.3v nets to PSUs and not Edison; removed tantalum caps; replaced LDO Vout caps with MLCCs and series ESRs; laid out board and ready to route
Parts:
- added R20, R21: 1 Ohm, rcl:R-US_R0402
- C1, C3: device rcl:C-USC0402K -> rcl:C-USC0603K
- C14, C17: value 22uF TANT -> 22uF; device SparkFun-Capacitors:CAP_POL3528 -> rcl:C-USC0603K
- C24: value 470uF TANT -> 470uF; device SparkFun-Capacitors:CAP_POL3528 -> SparkFun-Capacitors:CAP_POLE
Connections:
- removed net 3.3V_2A: C14.+, C24.+, CN1.+3.3AUX@52, CN1.+3.3VAUX@2, CN1.+3.3VAUX@24, CN1.+3.3VAUX@39, CN1.+3.3VAUX@41, U3.OUT
- new net N$16: C17.1, R20.1
- new net N$21: C14.1, R21.1
- new net P$1: R20.2, U7.OUT
- net 1.5V: no longer C17.+, U7.OUT
- net 3.3V: now also C24.+, CN1.+3.3AUX@52, CN1.+3.3VAUX@2, CN1.+3.3VAUX@24, CN1.+3.3VAUX@39, CN1.+3.3VAUX@41, R21.2, U3.OUT; no longer U1.3.3V@1, U1.3.3V@2
- net GND: now also C14.2, C17.2; no longer C14.-, C17.-
Other:
- note added: "0.3"
- note added: "Changed: tants to MLCC/Elec; changed cap packages; removed Eddie 3.3v"
- note added: "Decoupling cap for pin 15"
- note added: "Each 0.1uF decoupling cap should be close to pins 23, 15, 5, 10, 29, 36"
- note removed: "0.2"
- note removed: "Changed: crystal footprint; DN_USB to AB; Mov. cap bank; rem. SJ"
- note removed: "Each 0.1uF filtering cap should be close to pins 23, 15, 5, 10, 29, 36"
- note removed: "Filtering cap for pin 15"
- moved on the sheet: C15, C24, C29, C7, U3, U7
